File: Pekaway_rework.kicad_sch (KiCad schematic)
At the start: 23 parts, among them J3 Conn_01x01_Socket, J4 Conn_01x01_Socket, J5 Conn_01x12_Socket, SW1 SW_Push

Commit message: init commit
Other:
- moved on the sheet: D1, D10, D11, D12, D2, D3, D4, D5, D6, D7, D8, D9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
