File: Pekaway_rework.kicad_pcb (KiCad board)
At the start: 2 copper layers, 104.5 x 79 mm, 23 parts, among them J3 Conn_01x01_Socket, J4 Conn_01x01_Socket, J5 Conn_01x12_Socket, SW1 SW_Push

Commit message: init commit
Routing:
- net Net-(D10-K): track 123.8 -> 122.0 mm
Changed lines of the file:
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@@
 	)
 	(segment
-		(start 159.5 51.5)
-		(end 159.5 40)
+		(start 142.2175 47.4)
+		(end 146.4 47.4)
+		(width 0.2)
+		(layer "F.Cu")
+		(net 10)
+	)
+	(segment
+		(start 142.2175 47.4)
+		(end 142.2175 56.9)
+		(width 0.2)
+		(layer "F.Cu")
+		(net 10)
+	)
+	(segment
+		(start 146.4 47.4)
+		(end 151.5 52.5)
 		(width 0.2)
 		(layer "F.Cu")
@@
 	)
 	(segment
-		(start 142.2175 47.4)
-		(end 142.2175 56.9)
+		(start 142.2875 47.47)
+		(end 142.2175 47.4)
+		(width 0.2)
+		(layer "F.Cu")
+		(net 10)
+	)
+	(segment
+		(start 164 38.5)
+		(end 173 38.5)
+		(width 0.2)
+		(layer "F.Cu")
+		(net 10)
+	)
+	(segment
+		(start 142.2875 101)
+		(end 142.2875 47.47)
+		(width 0.2)
+		(layer "F.Cu")
+		(net 10)
+	)
+	(segment
+		(start 162 40.5)
+		(end 164 38.5)
+		(width 0.2)
+		(layer "F.Cu")
+		(net 10)
+	)
+	(segment
+		(start 158.5 52.5)
+		(end 162 49)
+		(width 0.2)
+		(layer "F.Cu")
+		(net 10)
+	)
+	(segment
+		(start 151.5 52.5)
+		(end 158.5 52.5)
+		(width 0.2)
+		(layer "F.Cu")
+		(net 10)
+	)
+	(segment
+		(start 162 49)
+		(end 162 40.5)
+		(width 0.2)
+		(layer "F.Cu")
+		(net 10)
+	)
+	(segment
+		(start 176 46)
+		(end 176 52.5)
 		(width 0.2)
 		(layer "F.Cu")
@@
 		(start 176 41.5)
 		(end 176 46)
-		(width 0.2)
-		(layer "F.Cu")
-		(net 10)
-	)
-	(segment
-		(start 146.4 47.4)
-		(end 151.5 52.5)
-		(width 0.2)
-		(layer "F.Cu")
-		(net 10)
-	)
-	(segment
-		(start 159.5 40)
-		(end 161 38.5)
-		(width 0.2)
-		(layer "F.Cu")
-		(net 10)
-	)
-	(segment
-		(start 142.2875 47.47)
-		(end 142.2175 47.4)
-		(width 0.2)
-		(layer "F.Cu")
-		(net 10)
-	)
-	(segment
-		(start 142.2875 101)
-		(end 142.2875 47.47)
-		(width 0.2)
-		(layer "F.Cu")
-		(net 10)
-	)
-	(segment
-		(start 151.5 52.5)
-		(end 158.5 52.5)
-		(width 0.2)
-		(layer "F.Cu")
-		(net 10)
-	)
-	(segment
-		(start 158.5 52.5)
-		(end 159.5 51.5)
-		(width 0.2)
-		(layer "F.Cu")
-		(net 10)
-	)
-	(segment
-		(start 176 46)
-		(end 176 52.5)
-		(width 0.2)
-		(layer "F.Cu")
-		(net 10)
-	)
-	(segment
-		(start 142.2175 47.4)
-		(end 146.4 47.4)
-		(width 0.2)
-		(layer "F.Cu")
-		(net 10)
-	)
-	(segment
-		(start 161 38.5)
-		(end 173 38.5)
 		(width 0.2)
 		(layer "F.Cu")
@@
 			(clearance 0.5)
 		)
-		(min_thickness 0.25)
+		(min_thickness 0.5)
 		(filled_areas_thickness no)
 		(fill yes
@@
 			(pts
 				(xy 152.500016 52) (xy 158.5 52) (xy 158.5 43) (xy 155.5 39.5) (xy 129.5 39.5) (xy 112 50.5) (xy 112 54)
-				(xy 113 55) (xy 124.230774 55) (xy 135 49) (xy 135 49) (xy 135 49) (xy 150.750016 49)
-			)
-		)
+				(xy 113 55) (xy 124.230774 55) (xy 135 49) (xy 150.750016 49)
+			)
+		)

Commit message: exported gerbers
Other:
- board text removed: "- Montage löcher hinzufügen - Leiterbahn dicke beachten!!! - Beschriftung für zusammenhängende Kanäle - Sicherungen zusammenfassen in zweier Gruppen"
Changed lines of the file:
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@@
 			(outputformat 1)
 			(mirror no)
-			(drillshape 1)
+			(drillshape 0)
 			(scaleselection 1)
-			(outputdirectory "")
+			(outputdirectory "gerbers/")
 		)
 	)
@@
 		(layer "Edge.Cuts")
 	)
-	(gr_text "- Montage löcher hinzufügen\n- Leiterbahn dicke beachten!!!\n- Beschriftung für zusammenhängende Kanäle\n- Sicherungen zusammenfassen in zweier Gruppen"
-		(at 123.5 129 0)
-		(layer "F.Cu")
-		(effects
-			(font
-				(size 1.5 1.5)
-				(thickness 0.3)
-				(bold yes)
-			)
-			(justify left bottom)
-		)
-	)
 	(gr_text "GND_1"
